File: motor-controller/motor-controller.kicad_sch (KiCad schematic)
At the start: 20 parts

Commit message: Add in a lot of other stuff hehe
Parts:
- removed J?: SCREW MOTOR B, symbol Connector:Screw_Terminal_01x01
- removed Q? (x2): Q_NMOS_DGS, symbol Device:Q_NMOS_DGS
- removed R? (x2): 10k, symbol Device:R_US
- removed R? (x2): 4.7, symbol Device:R_US
- added C? (x2): 1uF, symbol Device:C_Small
- added C? (x2): 0.1uF, symbol Device:C_Small
- added D? (x2): D_Schottky, symbol Device:D_Schottky
- added D?: PWR LED, symbol Device:LED
- added J?: SCREW MOTOR B, symbol Connector:Screw_Terminal_01x01
- added Q? (x2): Q_NMOS_DGS, symbol Device:Q_NMOS_DGS
- added R? (x2): 4.7, symbol Device:R_US
- added R?: 1k, symbol Device:R_US
- added R? (x2): 10k, symbol Device:R_US
- added TP? (x4): TestPoint, symbol Connector:TestPoint
- added U? (x2): IR2301, symbol Driver_FET:IR2301
Connections:
- net GATE_A_HIGH: now also TP?.1, U?.7 (HO)
- net GATE_A_LOW: now also TP?.1, U?.5 (LO)
- net GND: now also C?.2, C?.2, D?.1 (K), Q?.3 (S), R?.1, R?.1, U?.4 (COM), U?.4 (COM)
- net MOTOR_A: now also C?.2, U?.6 (VS)
- net MOTOR_B: now also C?.2, J?.1 (Pin_1), Q?.1 (D), Q?.3 (S), U?.6 (VS)
- net VBUS: now also C?.1, C?.1, D?.2 (A), D?.2 (A), Q?.1 (D), R?.1, U?.1 (VCC), U?.1 (VCC)
- new net: C?.1, D?.1 (K), U?.8 (VB) (x2)
- new net: D?.2 (A), R?.2
- new net: Q?.2 (G), R?.2 (x2)
- new net GATE_B_HIGH: R?.1, R?.2, TP?.1, U?.7 (HO)
- new net GATE_B_LOW: R?.1, R?.2, TP?.1, U?.5 (LO)
- new net PWM_A_HIGH: U?.2 (HIN)
- new net PWM_A_LOW: U?.3 (LIN)
- new net PWM_B_HIGH: U?.2 (HIN)
- new net PWM_B_LOW: U?.3 (LIN)
Other:
- added sheet controller (controller.kicad_sch)
- moved on the sheet: C?, J?, Q?, R?

Commit message: Add in some more footprints and components
Parts:
- removed D?: PWR LED, symbol Device:LED
- removed Q? (x4): Q_NMOS_DGS, symbol Device:Q_NMOS_DGS
- removed R?: 1k, symbol Device:R_US
- added Q? (x4): MCU80N03-TP, Package_TO_SOT_SMD:TO-252-3_TabPin2, symbol Device:Q_NMOS_GDS
- C? (x3): footprint (none) -> motor-controller-footprints:CP_Elec_12.5x13.5; Digikey Part Num (none) -> 565-2480-1-ND
- C? (x2): footprint (none) -> Capacitor_SMD:C_0805_2012Metric_Pad1.18x1.45mm_HandSolder; Digikey Part Num (none) -> 1276-6470-1-ND
- C? (x2): footprint (none) -> Capacitor_SMD:C_0603_1608Metric_Pad1.08x0.95mm_HandSolder; Digikey Part Num (none) -> 399-14105-1-ND
- C?: footprint (none) -> Capacitor_SMD:C_1206_3216Metric_Pad1.33x1.80mm_HandSolder; Digikey Part Num (none) -> 1276-6736-1-ND
- D? (x2): footprint (none) -> Diode_SMD:D_SMB; Digikey Part Num (none) -> 497-12627-1-ND
- R? (x4): footprint (none) -> Resistor_SMD:R_0603_1608Metric_Pad0.98x0.95mm_HandSolder; Digikey Part Num (none) -> 1276-3485-1-ND
- R? (x4): footprint (none) -> Resistor_SMD:R_0603_1608Metric_Pad0.98x0.95mm_HandSolder; Digikey Part Num (none) -> RNCP0603FTD4R70CT-ND
- TP? (x4): footprint (none) -> TestPoint:TestPoint_Pad_D1.0mm
- U? (x2): footprint (none) -> Package_SO:SOIC-8-N7_3.9x4.9mm_P1.27mm
Connections:
- net GND: now also Q?.3 (S), Q?.3 (S)
- net MOTOR_A: now also Q?.2 (D), Q?.3 (S)
- net MOTOR_B: now also Q?.2 (D), Q?.3 (S)
- net VBUS: now also Q?.2 (D), Q?.2 (D)
- net at R?.2: now also Q?.1 (G) (x4)

Commit message: first stab at placement
Parts:
- removed C? (x2): 470uF, motor-controller-footprints:CP_Elec_12.5x13.5, symbol Device:C_Polarized_Small_US
- added H1, H2, H3, H4: MountingHole, MountingHole:MountingHole_2.1mm, symbol Mechanical:MountingHole
- D1, D2: renamed from D?; value D_Schottky -> STPS130U
- J1, J2, J3, J4: renamed from J?; footprint (none) -> motor-controller-footprints:7698-SEMS; Digikey Part Num (none) -> 36-7698-SEMS-ND
- U1, U2: renamed from U?; footprint Package_SO:SOIC-8-N7_3.9x4.9mm_P1.27mm -> Package_SO:SOIC-8_3.9x4.9mm_P1.27mm
- gave numbers to parts that had none: 22
Other:
- moved on the sheet: C6
