File: motor-controller/motor-controller.kicad_sch (KiCad schematic)
At the start: 34 parts, among them J1 SCREW +, J2 SCREW -, J3 SCREW MOTOR A, J4 SCREW MOTOR B, Q1 MCU80N03-TP, Q2 MCU80N03-TP, Q3 MCU80N03-TP, Q4 MCU80N03-TP, U1 IR2301, U2 IR2301

Commit message: Stuff
Parts:
- added H5: Logo, motor-controller-footprints:basiliskLogo, symbol Mechanical:MountingHole
Changed lines of the file:
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@@
     (pin "1")
+  )
+  (symbol (lib_id "Mechanical:MountingHole") (at 168.91 193.04 0) (unit 1)
+    (in_bom yes) (on_board yes) (fields_autoplaced)
+    (property "Reference" "H5" (id 0) (at 171.45 192.1315 0)
+      (effects (font (size 1.27 1.27)) (justify left))
+    )
+    (property "Value" "Logo" (id 1) (at 171.45 194.9066 0)
+      (effects (font (size 1.27 1.27)) (justify left))
+    )
+    (property "Footprint" "motor-controller-footprints:basiliskLogo" (id 2) (at 168.91 193.04 0)
+      (effects (font (size 1.27 1.27)) hide)
+    )
+    (property "Datasheet" "~" (id 3) (at 168.91 193.04 0)
+      (effects (font (size 1.27 1.27)) hide)
+    )
   )
   (symbol (lib_id "power:GND") (at 121.92 130.81 0) (unit 1)
@@
       (reference "H4") (unit 1) (value "2mm") (footprint "MountingHole:MountingHole_2.1mm")
     )
+    (path "/bc8c29c1-b6ef-4c77-b66c-bd2bfce1bc73"
+      (reference "H5") (unit 1) (value "Logo") (footprint "motor-controller-footprints:basiliskLogo")
+    )
     (path "/54351f28-c2d1-4914-b8a7-3b991e3c2026"
