File: motor-controller/motor-controller.kicad_sch (KiCad schematic)
At the start: 26 parts, among them J1 SCREW +, J2 SCREW -, J3 SCREW MOTOR A, J4 SCREW MOTOR B, Q1 EPC2206, Q2 EPC2206, Q3 EPC2206, Q4 EPC2206, U1 uP1966E, U2 uP1966E

Commit message: Update hardware
Parts:
- removed H4: 2mm, MountingHole:MountingHole_2.1mm, symbol Mechanical:MountingHole
- removed Q1, Q2, Q3, Q4: EPC2206, eec:EPC-EPC2206-MFG, symbol GaN FET:EPC2206
- removed U1, U2: uP1966E, motor-controller-footprints:uP1966E, symbol basilisk_libs:uP1966E
- added C14, C16, C4: 10uF, Capacitor_SMD:C_1206_3216Metric_Pad1.33x1.80mm_HandSolder, symbol Device:C_Small
- added D1, D2: PMEG3005AESFYL, Diode_SMD:D_0603_1608Metric_Pad1.05x0.95mm_HandSolder, symbol Device:D_Schottky
- added Q1, Q2, Q3, Q4: AOD4132, Package_TO_SOT_SMD:TO-252-2, symbol Device:Q_NMOS_GDS
- added R1, R2, R3, R4: 4.7, Resistor_SMD:R_0603_1608Metric_Pad0.98x0.95mm_HandSolder, symbol Device:R_US
- added U1, U2: IRS2301S, Package_SO:SOIC-8_3.9x4.9mm_P1.27mm, symbol Driver_FET:IRS2301S
- C1, C17, C2: Digikey Part Num 399-14105-1-ND -> 1276-CL10B104KB8NNNLCT-ND
- C15, C3, C5, C6, C7, C8: footprint Capacitor_SMD:C_1206_3216Metric -> Capacitor_SMD:C_1206_3216Metric_Pad1.33x1.80mm_HandSolder
- C18: value 0.1uF -> 10uF; footprint Capacitor_SMD:C_0603_1608Metric_Pad1.08x0.95mm_HandSolder -> Capacitor_SMD:C_1206_3216Metric_Pad1.33x1.80mm_HandSolder; Digikey Part Num 399-14105-1-ND -> 1276-6736-1-ND
- C9: value 10uF -> 0.1uF; footprint Capacitor_SMD:C_1206_3216Metric -> Capacitor_SMD:C_0603_1608Metric_Pad1.08x0.95mm_HandSolder; Digikey Part Num 1276-6736-1-ND -> 1276-CL10B104KB8NNNLCT-ND
- J3: value SCREW MOTOR A -> SCREW +
- J4: value SCREW MOTOR B -> SCREW -
Connections:
- net +5V is gone; now on net VBUS: C1.1, C18.1
- net GND: now also C17.2, C14.2, C16.2, C4.2, Q2.3 (S), Q4.3 (S), U1.4 (COM), U2.4 (COM); no longer C9.2
- net PWM_A_HIGH: now also U1.2 (HIN)
- net PWM_A_LOW: now also U1.3 (LIN)
- net PWM_B_HIGH: now also U2.2 (HIN)
- net PWM_B_LOW: now also U2.3 (LIN)
- net VBUS: now also C17.1, C14.1, C16.1, C4.1, D1.2 (A), D2.2 (A), Q1.2 (D), Q3.2 (D), U1.1 (VCC), U2.1 (VCC); no longer C9.1
- net SW_A: now reaches C2.2
- net SW_A: now also J3.1 (Pin_1), Q1.3 (S), Q2.2 (D), U1.6 (VS)
- net PHASE A: no longer names the net of C2.1
- net PHASE A: now also D1.1 (K), U1.8 (VB); no longer J3.1 (Pin_1)
- net PHASE B renamed SW_B
- net SW_B: now also C9.2, Q3.3 (S), Q4.2 (D), U2.6 (VS); no longer C17.1
- new net: R1.1, U1.7 (HO)
- new net: Q1.1 (G), R1.2
- new net: Q3.1 (G), R3.2
- new net: C9.1, D2.1 (K), U2.8 (VB)
- new net: R2.1, U1.5 (LO)
- new net: R3.1, U2.7 (HO)
- new net: R4.1, U2.5 (LO)
- new net: Q4.1 (G), R4.2
- new net: Q2.1 (G), R2.2
- no-connect marks 2 -> 0
Other:
- moved on the sheet: J1, J2
