File: motor-controller/motor-controller.kicad_pcb (KiCad board)
At the start: 2 copper layers, 33.5 x 83.8 mm, 54 parts, among them J1 SCREW +, J2 SCREW -, J3 SCREW MOTOR A, J4 SCREW MOTOR B, J5 Conn_01x05, J6 Conn_01x03, Q1 MCU80N03-TP, Q2 MCU80N03-TP, Q3 MCU80N03-TP, Q4 MCU80N03-TP, U1 IR2301, U2 IR2301, U3 TC1047xNB, U4 STM32G030F6P6TR, U5 NCP1117ST33T3G, U6 LM78M05

Commit message: More layout stuff
Parts:
- moved D3 1.14 mm to (141.2, 151.4)
- moved R10 1.14 mm to (143.9, 149.1)
- moved R11 1.14 mm to (141.2, 148.2)
- moved R9 1.14 mm to (141.2, 154.6)
- moved R14 1.14 mm to (143.9, 153.7)
- moved D2 1.02 mm to (143.8, 141.7)
- moved U2 1.02 mm to (148.8, 141.7)
- moved C2 1.02 mm to (148.1, 146.8)
- moved C4 1.02 mm to (152.8, 140.3)
- moved C7 1.02 mm to (147.8, 137.2)
- moved Q2 0.58 mm to (159.4, 124.8)
- moved Q3 0.58 mm to (144.3, 124.8)
- moved Q4 0.58 mm to (151.9, 124.8)
- moved R2 0.58 mm to (159.4, 132.4)
- moved R3 0.58 mm to (164.5, 132.4)
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
Commit message: Stuff
Parts:
- added H5: Logo, motor-controller-footprints:basiliskLogo, B.Cu at (155.4, 160.0)
- H1, H2, H3, H4: value MountingHole -> 2mm
- moved D3 0.51 mm to (141.7, 151.4)
- moved R10 0.51 mm to (144.4, 149.1)
- moved R11 0.51 mm to (141.7, 148.2)
- moved R9 0.51 mm to (141.7, 154.6)
- moved R14 0.51 mm to (144.4, 153.7)
- moved R3 0.35 mm to (164.9, 132.4)
- moved TP1 0.35 mm to (165.4, 135.5)
- moved Q1 0.35 mm to (167.1, 124.9)
- moved Q2 0.35 mm to (159.8, 124.8)
- moved R1 0.35 mm to (167.1, 132.4)
- moved R2 0.35 mm to (159.8, 132.4)
- moved R4 0.35 mm to (157.5, 132.4)
- moved TP2 0.35 mm to (158.3, 135.5)
- moved R5 0.15 mm to (142.0, 132.4)
- moved R7 0.07 mm to (144.3, 132.4)
Routing:
- net +3V3: track 0.00 -> 99.0 mm, vias 0 -> 5
- net VBUS: track 0.00 -> 43.0 mm, vias 0 -> 13
- net +5V: track 0.00 -> 38.5 mm, vias 0 -> 1
- net /controller/ANALOG_TEMP: track 0.00 -> 33.8 mm, vias 0 -> 2
- net PWM_A_LOW: track 0.00 -> 28.4 mm
- net PWM_A_HIGH: track 0.00 -> 26.9 mm
- net PWM_B_HIGH: track 0.00 -> 25.6 mm, vias 0 -> 2
- net PWM_B_LOW: track 0.00 -> 24.3 mm, vias 0 -> 2
- net /controller/LED_G: track 0.00 -> 23.0 mm, vias 0 -> 2
- net GND: track 0.00 -> 19.6 mm, vias 0 -> 23
- net /controller/LED_B: track 0.00 -> 18.7 mm, vias 0 -> 2
- net /controller/PWM_IN: track 0.00 -> 18.2 mm
- net /GATE_A_LOW: track 0.00 -> 17.5 mm, vias 0 -> 2
- net /controller/LED_R: track 0.00 -> 15.2 mm
- net /GATE_B_HIGH: track 0.00 -> 13.3 mm
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- added copper zone on B.Cu, net /MOTOR_A
- added copper zone on F.Cu, net /MOTOR_A
- added copper zone on In2.Cu, net /MOTOR_A
- added copper zone on F.Cu, net /MOTOR_B
- added copper zone on In2.Cu, net /MOTOR_B
- added copper zone on F.Cu, net GND
- added copper zone on In1.Cu, net GND
- added copper zone on F.Cu, net VBUS
- added copper zone on In2.Cu, net VBUS
Other:
- copper layers 2 -> 4
- board text added: "Sahil Kale Samson Hua Rev 1.0 1/15/2022"

Commit message: Minor trace change and add STEP file
Routing:
- added copper zone on B.Cu, net VBUS
Changed lines of the file:
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@@
+    (effects (font (size 1.5 1.5) (thickness 0.3)))
+  )
+  (gr_text "+" (at 169.164 115.316) (layer "F.SilkS")
+    (effects (font (size 1.5 1.5) (thickness 0.3)))
+  )
+  (gr_text "-" (at 141.732 115.316) (layer "F.SilkS")
     (effects (font (size 1.5 1.5) (thickness 0.3)))
   )
@@
   (segment (start 146.59855 139.59745) (end 146.939 139.257) (width 0.381) (layer "F.Cu") (net 5))
   (segment (start 143.765403 139.59745) (end 146.59855 139.59745) (width 0.381) (layer "F.Cu") (net 5))
-  (segment (start 146.552 130.804) (end 147.32 131.572) (width 0.2032) (layer "F.Cu") (net 6))
-  (segment (start 148.336 137.103717) (end 148.336 131.572) (width 0.2032) (layer "F.Cu") (net 6))
   (segment (start 146.552 129.038065) (end 146.552 130.804) (width 0.2032) (layer "F.Cu") (net 6))
+  (segment (start 146.552 133.344) (end 146.552 130.804) (width 0.25) (layer "F.Cu") (net 6))
   (segment (start 149.479 137.9485) (end 148.6905 137.16) (width 0.2032) (layer "F.Cu") (net 6))
-  (segment (start 147.32 131.572) (end 148.336 131.572) (width 0.2032) (layer "F.Cu") (net 6))
+  (segment (start 148.6905 135.4825) (end 146.552 133.344) (width 0.25) (layer "F.Cu") (net 6))
+  (segment (start 148.6905 137.16) (end 148.6905 135.4825) (width 0.25) (layer "F.Cu") (net 6))
   (segment (start 149.479 139.257) (end 149.479 137.9485) (width 0.2032) (layer "F.Cu") (net 6))
   (via (at 150.876 118.364) (size 0.8) (drill 0.4) (layers "F.Cu" "B.Cu") (free) (net 6))
@@
     )
   )
-  (zone (net 1) (net_name "VBUS") (layer "In2.Cu") (hatch edge 0.508)
+  (zone (net 1) (net_name "VBUS") (layers "In2.Cu" "B.Cu") (hatch edge 0.508)
     (connect_pads (clearance 0.508))
     (min_thickness 0.254) (filled_areas_thickness no)
