File: motor-controller/motor-controller.kicad_pcb (KiCad board)
At the start: 4 copper layers, 30.5 x 51.3 mm, 43 parts, among them J1 SCREW +, J2 SCREW -, J3 SCREW MOTOR A, J4 SCREW MOTOR B, J5 Conn_01x05, J6 Conn_01x03, Q1 EPC2206, Q2 EPC2206, Q3 EPC2206, Q4 EPC2206, U1 uP1966E, U2 uP1966E, U4 STM32G030F6P6TR, U5 NCP1117ST33T3G, U6 LM78M05

Commit message: Add in released stuff
Routing:
- net VBUS: track 41.4 -> 42.3 mm
- net PWM_B_LOW: track 16.6 -> 17.3 mm
- net PWM_B_HIGH: track 15.0 -> 15.6 mm

Commit message: Update hardware
Parts:
- removed H4: 2mm, MountingHole:MountingHole_2.1mm
- added C14: 10uF, Capacitor_SMD:C_1206_3216Metric_Pad1.33x1.80mm_HandSolder, F.Cu at (146.1, 151.9)
- added C16: 10uF, Capacitor_SMD:C_1206_3216Metric_Pad1.33x1.80mm_HandSolder, F.Cu at (168.9, 158.5)
- added C4: 10uF, Capacitor_SMD:C_1206_3216Metric_Pad1.33x1.80mm_HandSolder, F.Cu at (168.9, 151.6)
- added D1: PMEG3005AESFYL, Diode_SMD:D_0603_1608Metric_Pad1.05x0.95mm_HandSolder, F.Cu at (149.9, 158.0)
- added D2: PMEG3005AESFYL, Diode_SMD:D_0603_1608Metric_Pad1.05x0.95mm_HandSolder, F.Cu at (159.0, 157.7)
- added R1: 4.7, Resistor_SMD:R_0603_1608Metric_Pad0.98x0.95mm_HandSolder, F.Cu at (145.6, 149.3)
- added R2: 4.7, Resistor_SMD:R_0603_1608Metric_Pad0.98x0.95mm_HandSolder, F.Cu at (150.6, 149.3)
- added R3: 4.7, Resistor_SMD:R_0603_1608Metric_Pad0.98x0.95mm_HandSolder, F.Cu at (164.8, 149.3)
- added R4: 4.7, Resistor_SMD:R_0603_1608Metric_Pad0.98x0.95mm_HandSolder, F.Cu at (159.5, 149.3)
- C15, C3, C5, C6, C7, C8: footprint Capacitor_SMD:C_1206_3216Metric -> Capacitor_SMD:C_1206_3216Metric_Pad1.33x1.80mm_HandSolder
- C18: value 0.1uF -> 10uF; footprint Capacitor_SMD:C_0603_1608Metric_Pad1.08x0.95mm_HandSolder -> Capacitor_SMD:C_1206_3216Metric_Pad1.33x1.80mm_HandSolder
- C9: value 10uF -> 0.1uF; footprint Capacitor_SMD:C_1206_3216Metric -> Capacitor_SMD:C_0603_1608Metric_Pad1.08x0.95mm_HandSolder
- J3: value SCREW MOTOR A -> SCREW +
- J4: value SCREW MOTOR B -> SCREW -
- Q1, Q2, Q3, Q4: value EPC2206 -> AOD4132; footprint eec:EPC-EPC2206-MFG -> Package_TO_SOT_SMD:TO-252-2
- U1, U2: value uP1966E -> IRS2301S; footprint motor-controller-footprints:uP1966E -> Package_SO:SOIC-8_3.9x4.9mm_P1.27mm
- moved H5 25.5 mm to (157.2, 140.5)
- moved C6 23.5 mm to (168.9, 160.8), turned to 0 degrees
- moved C8 20.0 mm to (146.1, 159.0)
- moved C3 19.7 mm to (146.0, 154.4)
- moved C15 19.3 mm to (146.1, 156.7)
- moved C9 15.7 mm to (161.5, 151.6), turned to 0 degrees
- moved Q3 14.3 mm to (167.9, 143.0)
- moved J4 12.7 mm to (160.1, 128.1)
- moved J3 12.7 mm to (149.6, 128.1)
- moved H1 12.4 mm to (169.7, 128.8)
- moved H3 12.4 mm to (144.3, 128.8)
- moved Q1 11.8 mm to (146.6, 143.0)
- moved Q2 10.7 mm to (153.7, 143.0)
- moved Q4 10.7 mm to (160.8, 143.0)
- moved C19 9.87 mm to (150.4, 165.4), turned to 0 degrees
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Connections:
- C1 pad 1: +5V -> VBUS
- C17 pad 1: /PHASE B -> VBUS
- C17 pad 2: Net-(C17-Pad2) -> GND
- C18 pad 1: +5V -> VBUS
- C2 pad 1: /PHASE A -> Net-(C2-Pad1)
- C2 pad 2: Net-(C2-Pad2) -> /SW_A
- C9 pad 1: VBUS -> Net-(C9-Pad1)
- C9 pad 2: GND -> /SW_B
- J3 pad 1: /PHASE A -> /SW_A
- J4 pad 1: /PHASE B -> /SW_B
- Q1 pad 2: /PHASE A -> VBUS
- Q1 pad 3: VBUS -> /SW_A
- Q2 pad 2: GND -> /SW_A
- Q2 pad 3: /PHASE A -> GND
- Q3 pad 2: /PHASE B -> VBUS
- Q3 pad 3: VBUS -> /SW_B
- Q4 pad 2: GND -> /SW_B
- Q4 pad 3: /PHASE B -> GND
- U4 pad 10: /controller/UART_RX -> unconnected-(U4-Pad10)
- U4 pad 9: /controller/UART_TX -> unconnected-(U4-Pad9)
- U5 pad 1: unconnected-(U5-Pad1) -> GND
Routing:
- net GND: track 51.0 -> 9.28 mm
- net +5V: track 54.6 -> 32.7 mm
- net VBUS: track 42.3 -> 20.7 mm, vias 40 -> 42
- net /SW_B: track 0.00 -> 21.1 mm
- net Net-(C2-Pad1): track 0.00 -> 11.1 mm
- net /PHASE B: track 10.5 -> 0.00 mm, vias 2 -> 0
- net /SW_A: track 0.00 -> 10.1 mm
- net /PHASE A: track 10.1 -> 0.00 mm, vias 2 -> 0
- net Net-(R3-Pad1): track 0.00 -> 9.46 mm
- net Net-(R2-Pad1): track 0.00 -> 8.34 mm
- net Net-(R1-Pad1): track 0.00 -> 8.29 mm
- net Net-(R4-Pad1): track 0.00 -> 6.58 mm
- net Net-(C9-Pad1): track 0.00 -> 5.92 mm
- net PWM_B_LOW: track 17.3 -> 22.9 mm
- net PWM_B_HIGH: track 15.6 -> 19.8 mm
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- added copper zone on F.Cu, net /SW_A
- added copper zone on F.Cu, net /SW_B
- removed copper zone on F.Cu, net /PHASE A
- removed copper zone on F.Cu, net /PHASE B
Other:
- board size 30.5 x 51.3 mm -> 30.5 x 63.8 mm
- board text added: "Sahil Kale Samson Hua Rev 1.2 | 4/1/22"
- board text removed: "Sahil Kale Samson Hua Rev 1.0 | 2/9/22"
