File: motor-controller/_autosave-motor-controller.kicad_pcb (KiCad board)
At the start: 4 copper layers, 30.5 x 51.3 mm, 43 parts, among them J1 SCREW +, J2 SCREW -, J3 SCREW MOTOR A, J4 SCREW MOTOR B, J5 Conn_01x05, J6 Conn_01x03, Q1 EPC2206, Q2 EPC2206, Q3 EPC2206, Q4 EPC2206, U1 uP1966E, U2 uP1966E, U4 STM32G030F6P6TR, U5 NCP1117ST33T3G, U6 LM78M05

Commit message: FInish layout
Changed lines of the file:
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@@
   (gr_line (start 169.672 138.684) (end 144.272 138.684) (layer "Edge.Cuts") (width 0.1))
   (gr_arc (start 144.272 189.992) (mid 142.475949 189.248051) (end 141.732 187.452) (layer "Edge.Cuts") (width 0.1))
-  (gr_text "Sahil Kale\nSamson Hua\nRev 1.0 | 2/9/22" (at 150.622 170.053) (layer "B.SilkS")
+  (gr_text "Sahil Kale\nSamson Hua\nRev 1.0 | 2/9/22" (at 150.368 171.704) (layer "B.SilkS")
     (effects (font (size 0.762 0.762) (thickness 0.15)) (justify mirror))
   )
@@
   (via (at 159.512 174.244) (size 0.4064) (drill 0.200406) (layers "F.Cu" "B.Cu") (net 27))
   (via (at 160.528 161.417) (size 0.4064) (drill 0.200406) (layers "F.Cu" "B.Cu") (net 27))
-  (segment (start 160.782 172.974) (end 159.512 174.244) (width 0.0889) (layer "B.Cu") (net 27))
-  (segment (start 160.528 161.544) (end 160.528 172.847) (width 0.0889) (layer "B.Cu") (net 27))
+  (segment (start 160.528 173.228) (end 160.528 161.544) (width 0.0889) (layer "B.Cu") (net 27))
+  (segment (start 159.512 174.244) (end 160.528 173.228) (width 0.0889) (layer "B.Cu") (net 27))
   (segment (start 151.4875 169.672) (end 151.4875 171.2575) (width 0.254) (layer "F.Cu") (net 35))
   (segment (start 151.4875 171.2575) (end 151.7 171.47) (width 0.254) (layer "F.Cu") (net 35))
