File: motor-controller/_autosave-motor-controller.kicad_sch (KiCad schematic)
At the start: 27 parts, among them J1 SCREW +, J2 SCREW -, J3 SCREW MOTOR A, J4 SCREW MOTOR B, Q1 EPC2206, Q2 EPC2206, Q3 EPC2206, Q4 EPC2206, U1 uP1966E, U2 uP1966E

Commit message: FInish layout
Parts:
- removed C16: 10uF, Capacitor_SMD:C_1206_3216Metric, symbol Device:C_Small
Changed lines of the file:
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@@
-    (stroke (width 0) (type default) (color 0 0 0 0))
-  )
-  (wire (pts (xy 154.94 33.02) (xy 154.94 38.1))
     (stroke (width 0) (type default) (color 0 0 0 0))
   )
@@
   )
   (wire (pts (xy 115.57 88.9) (xy 118.11 88.9))
-    (stroke (width 0) (type default) (color 0 0 0 0))
-  )
-  (wire (pts (xy 154.94 43.18) (xy 154.94 52.07))
     (stroke (width 0) (type default) (color 0 0 0 0))
   )
@@
     (pin "1")
   )
-  (symbol (lib_id "Device:C_Small") (at 154.94 40.64 0) (unit 1)
-    (in_bom yes) (on_board yes) (fields_autoplaced)
-    (property "Reference" "C16" (id 0) (at 157.2641 39.7378 0)
-      (effects (font (size 1.27 1.27)) (justify left))
-    )
-    (property "Value" "10uF" (id 1) (at 157.2641 42.5129 0)
-      (effects (font (size 1.27 1.27)) (justify left))
-    )
-    (property "Footprint" "Capacitor_SMD:C_1206_3216Metric" (id 2) (at 154.94 40.64 0)
-      (effects (font (size 1.27 1.27)) hide)
-    )
-    (property "Datasheet" "~" (id 3) (at 154.94 40.64 0)
-      (effects (font (size 1.27 1.27)) hide)
-    )
-    (property "Digikey Part Num" "1276-6736-1-ND" (id 4) (at 154.94 40.64 0)
-      (effects (font (size 1.27 1.27)) hide)
-    )
-    (pin "1")
-    (pin "2")
-  )
-  (symbol (lib_id "power:GND") (at 154.94 52.07 0) (unit 1)
-    (in_bom yes) (on_board yes) (fields_autoplaced)
-    (property "Reference" "#PWR0108" (id 0) (at 154.94 58.42 0)
-      (effects (font (size 1.27 1.27)) hide)
-    )
-    (property "Value" "GND" (id 1) (at 154.94 56.6325 0))
-    (property "Footprint" "" (id 2) (at 154.94 52.07 0)
-      (effects (font (size 1.27 1.27)) hide)
-    )
-    (property "Datasheet" "" (id 3) (at 154.94 52.07 0)
-      (effects (font (size 1.27 1.27)) hide)
-    )
-    (pin "1")
-  )
   (symbol (lib_id "power:GND") (at 114.3 52.07 0) (unit 1)
     (in_bom yes) (on_board yes) (fields_autoplaced)
@@
     (pin "2")
   )
-  (symbol (lib_id "power:VBUS") (at 154.94 33.02 0) (unit 1)
-    (in_bom yes) (on_board yes) (fields_autoplaced)
-    (property "Reference" "#PWR0111" (id 0) (at 154.94 36.83 0)
-      (effects (font (size 1.27 1.27)) hide)
-    )
-    (property "Value" "VBUS" (id 1) (at 154.94 29.4155 0))
-    (property "Footprint" "" (id 2) (at 154.94 33.02 0)
-      (effects (font (size 1.27 1.27)) hide)
-    )
-    (property "Datasheet" "" (id 3) (at 154.94 33.02 0)
-      (effects (font (size 1.27 1.27)) hide)
-    )
-    (pin "1")
-  )
   (symbol (lib_id "power:VBUS") (at 152.4 86.36 0) (mirror y) (unit 1)
     (in_bom yes) (on_board yes) (fields_autoplaced)
@@
       (reference "#PWR0107") (unit 1) (value "VBUS") (footprint "")
     )
-    (path "/1764d985-3276-44d4-9601-8161e4e5f363"
-      (reference "#PWR0108") (unit 1) (value "GND") (footprint "")
-    )
     (path "/b86dabc5-a078-41e9-9da0-7b7feda7d0a9"
       (reference "#PWR0109") (unit 1) (value "GND") (footprint "")
@@
       (reference "#PWR0110") (unit 1) (value "VBUS") (footprint "")
     )
-    (path "/cdc98f98-c59b-4184-901d-dc51bdcde9fa"
-      (reference "#PWR0111") (unit 1) (value "VBUS") (footprint "")
-    )
     (path "/2857d539-20d0-4a12-b8ce-7f075a7481fc"
       (reference "#PWR0112") (unit 1) (value "GND") (footprint "")
@@
       (reference "#PWR0119") (unit 1) (value "+3V3") (footprint "")
     )
-    (path "/a64d3074-4d79-49a2-86f7-39249c3118cd/ee4fcd8e-9cb9-44a0-b7b1-83a1a5a43353"
-      (reference "#PWR0120") (unit 1) (value "+3V3") (footprint "")
-    )
     (path "/a64d3074-4d79-49a2-86f7-39249c3118cd/a8b9a906-ebdd-405c-a29b-5d4111eb202e"
       (reference "#PWR0121") (unit 1) (value "GND") (footprint "")
     )
-    (path "/a64d3074-4d79-49a2-86f7-39249c3118cd/b5028a48-87d2-4b03-9592-e522058ec45e"
-      (reference "#PWR0122") (unit 1) (value "GND") (footprint "")
-    )
     (path "/a64d3074-4d79-49a2-86f7-39249c3118cd/88d74181-d443-4061-b810-8c9d38e5ab60"
       (reference "#PWR0123") (unit 1) (value "GND") (footprint "")
@@
       (reference "C13") (unit 1) (value "10uF") (footprint "Capacitor_SMD:C_0805_2012Metric_Pad1.18x1.45mm_HandSolder")
     )
-    (path "/a64d3074-4d79-49a2-86f7-39249c3118cd/397b5ee8-5e1a-484b-a460-f7a37a322fed"
-      (reference "C14") (unit 1) (value "0.1uF") (footprint "Capacitor_SMD:C_0603_1608Metric_Pad1.08x0.95mm_HandSolder")
-    )
     (path "/3e38b5c3-471d-4afe-95dd-e76c4c1efce5"
       (reference "C15") (unit 1) (value "10uF") (footprint "Capacitor_SMD:C_1206_3216Metric")
     )
-    (path "/0cc1900c-723b-4f29-9608-2a30b58df409"
-      (reference "C16") (unit 1) (value "10uF") (footprint "Capacitor_SMD:C_1206_3216Metric")
-    )
     (path "/9ca51022-3b91-44b5-80b7-5ad984fdfd44"
